Commit message: add code for differential drive movement of robile

File: robile_pybullet/robile3_config.urdf (robot description, URDF)
Before this commit: robot robile3_config, 19 links, 18 joints
Links:
- link robile_1_drive_left_hub_wheel_link: geometry collision cylinder length=0.035 radius=0.0515; visual mesh filename=file:///home/saiga/ros2_ws/install/robile_description/share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 scale=1 1 1
- link robile_1_drive_pivot_link: geometry collision box size=0.105 0.154 0.025; visual mesh filename=file:///home/saiga/ros2_ws/install/robile_description/share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 scale=1 1 1
- link robile_1_drive_right_hub_wheel_link: geometry collision cylinder length=0.035 radius=0.0515; visual mesh filename=file:///home/saiga/ros2_ws/install/robile_description/share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 scale=1 1 1
- link robile_1_link: geometry collision box size=0.233 0.233 0.239; visual mesh filename=file:///home/saiga/ros2_ws/install/robile_description/share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 scale=1 1 1
- link robile_2_drive_left_hub_wheel_link: geometry collision cylinder length=0.035 radius=0.0515; visual mesh filename=file:///home/saiga/ros2_ws/install/robile_description/share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 scale=1 1 1
- link robile_2_drive_pivot_link: geometry collision box size=0.105 0.154 0.025; visual mesh filename=file:///home/saiga/ros2_ws/install/robile_description/share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 scale=1 1 1
- link robile_2_drive_right_hub_wheel_link: geometry collision cylinder length=0.035 radius=0.0515; visual mesh filename=file:///home/saiga/ros2_ws/install/robile_description/share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 scale=1 1 1
- link robile_2_link: geometry collision box size=0.233 0.233 0.239; visual mesh filename=file:///home/saiga/ros2_ws/install/robile_description/share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 scale=1 1 1
- link robile_3_link: geometry collision box size=0.233 0.233 0.239; visual mesh filename=file:///home/saiga/ros2_ws/install/robile_description/share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 scale=1 1 1
- link robile_4_link: geometry collision box size=0.233 0.233 0.239; visual mesh filename=file:///home/saiga/ros2_ws/install/robile_description/share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 scale=1 1 1
- link robile_5_drive_left_hub_wheel_link: geometry collision cylinder length=0.035 radius=0.0515; visual mesh filename=file:///home/saiga/ros2_ws/install/robile_description/share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 scale=1 1 1
- link robile_5_drive_pivot_link: geometry collision box size=0.105 0.154 0.025; visual mesh filename=file:///home/saiga/ros2_ws/install/robile_description/share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 scale=1 1 1
- link robile_5_drive_right_hub_wheel_link: geometry collision cylinder length=0.035 radius=0.0515; visual mesh filename=file:///home/saiga/ros2_ws/install/robile_description/share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 scale=1 1 1
- link robile_5_link: geometry collision box size=0.233 0.233 0.239; visual mesh filename=file:///home/saiga/ros2_ws/install/robile_description/share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 scale=1 1 1
- link robile_6_drive_left_hub_wheel_link: geometry collision cylinder length=0.035 radius=0.0515; visual mesh filename=file:///home/saiga/ros2_ws/install/robile_description/share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 scale=1 1 1
- link robile_6_drive_pivot_link: geometry collision box size=0.105 0.154 0.025; visual mesh filename=file:///home/saiga/ros2_ws/install/robile_description/share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 scale=1 1 1
- link robile_6_drive_right_hub_wheel_link: geometry collision cylinder length=0.035 radius=0.0515; visual mesh filename=file:///home/saiga/ros2_ws/install/robile_description/share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 scale=1 1 1
- link robile_6_link: geometry collision box size=0.233 0.233 0.239; visual mesh filename=file:///home/saiga/ros2_ws/install/robile_description/share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 scale=1 1 1

Commit message: added base_laser_front_link to odom transfrom publisher

File: robile_pybullet/robile3_config.urdf (robot description, URDF)
Before this commit: robot robile3_config, 19 links, 18 joints
Links:
- link robile_1_drive_left_hub_wheel_link: geometry collision cylinder length=0.035 radius=0.0515; visual mesh filename=file:///home/sunesh/ros2_ws/install/robile_description/shar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 scale=1 1 1
- link robile_1_drive_pivot_link: geometry collision box size=0.105 0.154 0.025; visual mesh filename=file:///home/sunesh/ros2_ws/install/robile_description/shar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 scale=1 1 1
- link robile_1_drive_right_hub_wheel_link: geometry collision cylinder length=0.035 radius=0.0515; visual mesh filename=file:///home/sunesh/ros2_ws/install/robile_description/shar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 scale=1 1 1
- link robile_1_link: geometry collision box size=0.233 0.233 0.239; visual mesh filename=file:///home/sunesh/ros2_ws/install/robile_description/shar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 scale=1 1 1
- link robile_2_drive_left_hub_wheel_link: geometry collision cylinder length=0.035 radius=0.0515; visual mesh filename=file:///home/sunesh/ros2_ws/install/robile_description/shar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 scale=1 1 1
- link robile_2_drive_pivot_link: geometry collision box size=0.105 0.154 0.025; visual mesh filename=file:///home/sunesh/ros2_ws/install/robile_description/shar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 scale=1 1 1
- link robile_2_drive_right_hub_wheel_link: geometry collision cylinder length=0.035 radius=0.0515; visual mesh filename=file:///home/sunesh/ros2_ws/install/robile_description/shar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 scale=1 1 1
- link robile_2_link: geometry collision box size=0.233 0.233 0.239; visual mesh filename=file:///home/sunesh/ros2_ws/install/robile_description/shar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 scale=1 1 1
- link robile_3_link: geometry collision box size=0.233 0.233 0.239; visual mesh filename=file:///home/sunesh/ros2_ws/install/robile_description/shar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 scale=1 1 1
- link robile_4_link: geometry collision box size=0.233 0.233 0.239; visual mesh filename=file:///home/sunesh/ros2_ws/install/robile_description/shar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 scale=1 1 1
- link robile_5_drive_left_hub_wheel_link: geometry collision cylinder length=0.035 radius=0.0515; visual mesh filename=file:///home/sunesh/ros2_ws/install/robile_description/shar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 scale=1 1 1
- link robile_5_drive_pivot_link: geometry collision box size=0.105 0.154 0.025; visual mesh filename=file:///home/sunesh/ros2_ws/install/robile_description/shar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 scale=1 1 1
- link robile_5_drive_right_hub_wheel_link: geometry collision cylinder length=0.035 radius=0.0515; visual mesh filename=file:///home/sunesh/ros2_ws/install/robile_description/shar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 scale=1 1 1
- link robile_5_link: geometry collision box size=0.233 0.233 0.239; visual mesh filename=file:///home/sunesh/ros2_ws/install/robile_description/shar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 scale=1 1 1
- link robile_6_drive_left_hub_wheel_link: geometry collision cylinder length=0.035 radius=0.0515; visual mesh filename=file:///home/sunesh/ros2_ws/install/robile_description/shar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 scale=1 1 1
- link robile_6_drive_pivot_link: geometry collision box size=0.105 0.154 0.025; visual mesh filename=file:///home/sunesh/ros2_ws/install/robile_description/shar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 scale=1 1 1
- link robile_6_drive_right_hub_wheel_link: geometry collision cylinder length=0.035 radius=0.0515; visual mesh filename=file:///home/sunesh/ros2_ws/install/robile_description/shar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 scale=1 1 1
- link robile_6_link: geometry collision box size=0.233 0.233 0.239; visual mesh filename=file:///home/sunesh/ros2_ws/install/robile_description/shar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 scale=1 1 1
